Commit message: add map

File: src/robot_model/urdf/lidar.xacro (robot description, xacro)
@@ -4,5 +4,5 @@
         <parent link="chassis"/>
         <child link="laser_frame"/>
-        <origin xyz="0 0 0.17" rpy="0 0 0"/>
+        <origin xyz="0 0 0.27" rpy="0 0 0"/>
     </joint>
     <link name="laser_frame">

Commit message: add keyboard

File: src/robot_model/urdf/lidar.xacro (robot description, xacro)
@@ -4,5 +4,6 @@
         <parent link="chassis"/>
         <child link="laser_frame"/>
-        <origin xyz="0 0 0.27" rpy="0 0 0"/>
+        <origin xyz="0 0 0.23" rpy="0 0 0"/>
+        <!-- 0.27 -->
     </joint>
     <link name="laser_frame">
@@ -26,5 +27,5 @@
         <sensor name="laser" type="ray">
             <pose> 0 0 0 0 0 0 </pose>
-            <visualize>true</visualize>
+            <visualize>false</visualize>
             <update_rate>10</update_rate>
             <ray>

File: src/robot_model/urdf/robot.urdf.xacro (robot description, xacro)
@@ -5,3 +5,4 @@
     <xacro:include filename="gazebo_control.xacro" />
     <xacro:include filename="lidar.xacro" />
+    <xacro:include filename="gripper.xacro" />
 </robot>

File: src/robot_model/urdf/robot_core.xacro (robot description, xacro)
@@ -50,5 +50,5 @@
                 <cylinder length="0.15" radius="0.075"/>
             </geometry>
-            <material name="white"/>
+            <material name="pink"/>
         </visual>
         <collision>
@@ -65,5 +65,5 @@
     </link>
     <gazebo reference="chassis">
-        <material>Gazebo/White</material>
+        <material>Gazebo/Pink</material>
     </gazebo>
     <!-- Wheel Link -->
@@ -71,5 +71,5 @@
         <visual>
             <geometry>
-                <cylinder length="0.03" radius="0.07" />
+                <cylinder length="0.04" radius="0.08" />
             </geometry>
             <material name="blue"/>
@@ -77,18 +77,18 @@
         <collision>
             <geometry>
-                <cylinder length="0.03" radius="0.07" />
+                <cylinder length="0.04" radius="0.08" />
             </geometry>
         </collision>
-        <xacro:inertial_cylinder mass="0.1" length="0.03" radius="0.07">
+        <xacro:inertial_cylinder mass="0.1" length="0.04" radius="0.08">
             <origin xyz="0 0 0" rpy="0 0 0"/>
         </xacro:inertial_cylinder>
     </link>
     <gazebo reference="front_left_wheel">
-        <material>Gazebo/Blue</material>
+        <material>Gazebo/Red</material>
     </gazebo>
     <link name="front_right_wheel">
         <visual>
             <geometry>
-                <cylinder length="0.03" radius="0.07" />
+                <cylinder length="0.04" radius="0.08" />
             </geometry>
             <material name="red"/>
@@ -96,8 +96,8 @@
         <collision>
             <geometry>
-                <cylinder length="0.03" radius="0.07" />
+                <cylinder length="0.04" radius="0.08" />
             </geometry>
         </collision>
-        <xacro:inertial_cylinder mass="0.1" length="0.03" radius="0.07">
+        <xacro:inertial_cylinder mass="0.1" length="0.04" radius="0.08">
             <origin xyz="0 0 0" rpy="0 0 0"/>
         </xacro:inertial_cylinder>
@@ -109,5 +109,5 @@
         <visual>
             <geometry>
-                <cylinder length="0.03" radius="0.07" />
+                <cylinder length="0.04" radius="0.08" />
             </geometry>
             <material name="orange"/>
@@ -115,18 +115,18 @@
         <collision>
             <geometry>
-                <cylinder length="0.03" radius="0.07" />
+                <cylinder length="0.04" radius="0.08" />
             </geometry>
         </collision>
-        <xacro:inertial_cylinder mass="0.1" length="0.03" radius="0.07">
+        <xacro:inertial_cylinder mass="0.1" length="0.04" radius="0.08">
             <origin xyz="0 0 0" rpy="0 0 0"/>
         </xacro:inertial_cylinder>
     </link>
     <gazebo reference="back_left_wheel">
-        <material>Gazebo/Orange</material>
+        <material>Gazebo/Red</material>
     </gazebo>
     <link name="back_right_wheel">
         <visual>
             <geometry>
-                <cylinder length="0.03" radius="0.07" />
+                <cylinder length="0.04" radius="0.08" />
             </geometry>
             <material name="green"/>
@@ -134,13 +134,13 @@
         <collision>
             <geometry>
-                <cylinder length="0.03" radius="0.07" />
+                <cylinder length="0.04" radius="0.08" />
             </geometry>
         </collision>
-        <xacro:inertial_cylinder mass="0.1" length="0.03" radius="0.07">
+        <xacro:inertial_cylinder mass="0.1" length="0.04" radius="0.08">
             <origin xyz="0 0 0" rpy="0 0 0"/>
         </xacro:inertial_cylinder>
     </link>
     <gazebo reference="back_right_wheel">
-        <material>Gazebo/Green</material>
+        <material>Gazebo/Red</material>
     </gazebo>
     <!-- Wheel Joint -->
