Commit message: add gripperr

File: src/robot_model/urdf/gazebo_plugin.xacro (robot description, xacro)
@@ -4,5 +4,5 @@
         <gazebo>
             <plugin name="gazebo_ros2_control_robot" filename="libgazebo_ros2_control.so">
-                <parameters>$(find articubot_one)/config/velocity_controllers.yaml</parameters>
+                <parameters>$(find robot_model)/config/velocity_controllers.yaml</parameters>
             </plugin>
         </gazebo>

File: src/robot_model/urdf/gripper.xacro (robot description, xacro)
@@ -1,4 +1,4 @@
 <?xml version="1.0"?>
-<robot xmlns:xacro="http://www.ros.org/wiki/xacro" xmlns="http://www.ros.org/wiki/xacro">
+<robot xmlns:xacro="http://www.ros.org/wiki/xacro" >
     <!-- Gripper Base -->
     <link name="gripper_base">
@@ -11,53 +11,104 @@
         </visual>
         <collision>
+            <origin xyz="0 0 0" rpy="0 0 0"/>
             <geometry>
                 <box size="0.35 0.05 0.05"/>
             </geometry>
+            <surface>
+                <friction>
+                    <ode>
+                        <mu>2.0</mu>  <!-- Increase primary friction -->
+                        <mu2>2.0</mu2>  <!-- Increase secondary friction -->
+                    </ode>
+                </friction>
+                <contact>
+                    <ode>
+                        <restitution>0.0</restitution>  <!-- Lower the bounce factor -->
+                        <soft_cfm>0.1</soft_cfm>  <!-- Soft constraint for smooth contact -->
+                        <soft_erp>0.7</soft_erp>  <!-- Error reduction for smoother response -->
+                        <kp>1000.0</kp>  <!-- Reduce excessive force -->
+                        <kd>100.0</kd>  <!-- Damping to prevent sudden jumps -->
+                        <max_vel>0.01</max_vel>
+                    </ode>
+                </contact>
+            </surface>
         </collision>
-        <inertial>
-            <mass value="0.1"/>
+        <xacro:inertial_box mass="0.5" x="0.35" y="0.05" z="0.05" >
             <origin xyz="0 0 0" rpy="0 0 0"/>
-            <inertia ixx="0.01" ixy="0" ixz="0" iyy="0.01" iyz="0" izz="0.01"/>
-        </inertial>
+        </xacro:inertial_box>
     </link>
     <!-- Gripper Finger Left -->
     <link name="gripper_finger_left">
         <visual>
-            <origin xyz="-0.075 0 0" rpy="0 0 0"/>
+            <origin xyz="-0.075 -0.1 0" rpy="0 0 0"/>
             <geometry>
-                <box size="0.02 0.1 0.02"/>
+                <box size="0.0225 0.2 0.05"/>
             </geometry>
-            <material name="red"/>
+            <material name="orange"/>
         </visual>
         <collision>
+            <origin xyz="-0.075 -0.1 0" rpy="0 0 0"/>
             <geometry>
-                <box size="0.02 0.1 0.02"/>
+                <box size="0.0225 0.2 0.1"/>
             </geometry>
+            <surface>
+                <friction>
+                    <ode>
+                        <mu>2.0</mu>  <!-- Increase primary friction -->
+                        <mu2>2.0</mu2>  <!-- Increase secondary friction -->
+                    </ode>
+                </friction>
+                <contact>
+                    <ode>
+                        <restitution>0.0</restitution>  <!-- Lower the bounce factor -->
+                        <soft_cfm>0.1</soft_cfm>  <!-- Soft constraint for smooth contact -->
+                        <soft_erp>0.7</soft_erp>  <!-- Error reduction for smoother response -->
+                        <kp>1000.0</kp>  <!-- Reduce excessive force -->
+                        <kd>100.0</kd>  <!-- Damping to prevent sudden jumps -->
+                        <max_vel>0.01</max_vel>
+                    </ode>
+                </contact>
+            </surface>
         </collision>
-        <inertial>
-            <mass value="0.1"/>
-            <origin xyz="0 0 0" rpy="0 0 0"/>
-            <inertia ixx="0.001" ixy="0" ixz="0" iyy="0.001" iyz="0" izz="0.001"/>
-        </inertial>
+        <xacro:inertial_box mass="0.3" x="0.0225" y="0.2" z="0.05" >
+            <origin xyz="-0.075 -0.1 0" rpy="0 0 0"/>
+        </xacro:inertial_box>
     </link>
     <!-- Gripper Finger Right -->
     <link name="gripper_finger_right">
         <visual>
-            <origin xyz="0.075 0 0" rpy="0 0 0"/>
+            <origin xyz="0.075 -0.10 0" rpy="0 0 0"/>
             <geometry>
-                <box size="0.02 0.1 0.02"/>
+                <box size="0.0225 0.2 0.05"/>
             </geometry>
-            <material name="red"/>
+            <material name="orange"/>
         </visual>
         <collision>
+            <origin xyz="0.075 -0.10 0" rpy="0 0 0"/>
             <geometry>
-                <box size="0.02 0.1 0.02"/>
+                <box size="0.0225 0.2 0.1"/>
             </geometry>
+            <surface>
+                <friction>
+                    <ode>
+                        <mu>2.0</mu>  <!-- Increase primary friction -->
+                        <mu2>2.0</mu2>  <!-- Increase secondary friction -->
+                    </ode>
+                </friction>
+                <contact>
+                    <ode>
+                        <restitution>0.0</restitution>  <!-- Lower the bounce factor -->
+                        <soft_cfm>0.1</soft_cfm>  <!-- Soft constraint for smooth contact -->
+                        <soft_erp>0.7</soft_erp>  <!-- Error reduction for smoother response -->
+                        <kp>1000.0</kp>  <!-- Reduce excessive force -->
+                        <kd>100.0</kd>  <!-- Damping to prevent sudden jumps -->
+                        <max_vel>0.01</max_vel>
+                    </ode>
+                </contact>
+            </surface>
         </collision>
-        <inertial>
-            <mass value="0.1"/>
-            <origin xyz="0 0 0" rpy="0 0 0"/>
-            <inertia ixx="0.001" ixy="0" ixz="0" iyy="0.001" iyz="0" izz="0.001"/>
-        </inertial>
+        <xacro:inertial_box mass="0.3" x="0.0225" y="0.2" z="0.05" >
+            <origin xyz="0.075 -0.10 0" rpy="0 0 0"/>
+        </xacro:inertial_box>
     </link>
     <!-- Vertical Movement Joint for Gripper -->
@@ -65,8 +116,8 @@
         <parent link="chassis"/>
         <child link="gripper_base"/>
-        <origin xyz="0.25 0 0.05" rpy="0 0 1.57"/>
+        <origin xyz="0.25 0 0" rpy="0 0 1.57"/>
         <axis xyz="0 0 1"/>
-        <limit effort="10" lower="0" upper="0.13" velocity="0.1"/>
-        <dynamics damping="0.5" friction="0.1"/>
+        <limit effort="80" lower="0" upper="0.13" velocity="0.1"/>
+        <dynamics damping="50.0" friction="1.0"/>
     </joint>
     <!-- Gripper Finger Joints -->
@@ -74,29 +125,49 @@
         <parent link="gripper_base"/>
         <child link="gripper_finger_left"/>
-        <origin xyz="-0.075 -0.1 0" rpy="0 0 0"/>
+        <origin xyz="-0.075 0 0" rpy="0 0 0"/>
         <axis xyz="1 0 0"/>
-        <limit effort="10" lower="0" upper="0.1" velocity="0.1"/>
-        <dynamics damping="0.5" friction="0.1"/>
+        <limit effort="100" lower="0" upper="0.1" velocity="0.1"/>
+        <dynamics damping="20.0" friction="1.0"/>
     </joint>
     <joint name="gripper_finger_right_joint" type="prismatic">
         <parent link="gripper_base"/>
         <child link="gripper_finger_right"/>
-        <origin xyz="0.075 -0.1 0" rpy="0 0 0"/>
+        <origin xyz="0.075 0 0" rpy="0 0 0"/>
         <axis xyz="1 0 0"/>
-        <limit effort="10" lower="-0.1" upper="0" velocity="0.1"/>
-        <dynamics damping="0.5" friction="0.1"/>
+        <limit effort="100" lower="-0.1" upper="0" velocity="0.1"/>
+        <dynamics damping="20.0" friction="1.0"/>
     </joint>
     <!-- Gazebo Simulation for Gripper -->
     <gazebo reference="gripper_base">
-        <material>Gazebo/Pink</material>
+        <material>Gazebo/Gray</material>
         <gravity>true</gravity>
+        <ode>
+            <solver_iterations>500</solver_iterations>  <!-- Increase solver iterations -->
+            <solver_type>quick_nonlinear</solver_type>  <!-- Adjust solver for stability -->
+        </ode>
     </gazebo>
     <gazebo reference="gripper_finger_left">
-        <material>Gazebo/Red</material>
+        <material>Gazebo/Orange</material>
         <gravity>true</gravity>
+        <ode>
+            <solver_iterations>500</solver_iterations>  <!-- Increase solver iterations -->
+            <solver_type>quick_nonlinear</solver_type>  <!-- Adjust solver for stability -->
+        </ode>
+        <!-- <plugin name="gazebo_gripper" filename="libgazebo_ros_vacuum_gripper.so">
+            <always_on>true</always_on>
+            <topic>gripper/grasp</topic>
+        </plugin> -->
     </gazebo>
     <gazebo reference="gripper_finger_right">
-        <material>Gazebo/Red</material>
+        <material>Gazebo/Orange</material>
         <gravity>true</gravity>
+        <ode>
+            <solver_iterations>500</solver_iterations>  <!-- Increase solver iterations -->
+            <solver_type>quick_nonlinear</solver_type>  <!-- Adjust solver for stability -->
+        </ode>
+        <!-- <plugin name="gazebo_gripper" filename="libgazebo_ros_vacuum_gripper.so">
+            <always_on>true</always_on>
+            <topic>gripper/grasp</topic>
+        </plugin> -->
     </gazebo>
 </robot>
