Commit message: change material

File: src/robot_model/urdf/gripper.xacro (robot description, xacro)
@@ -140,5 +140,5 @@
     <!-- Gazebo Simulation for Gripper -->
     <gazebo reference="gripper_base">
-        <material>Gazebo/Gray</material>
+        <material>Gazebo/WoodPallet </material>
         <gravity>true</gravity>
         <ode>
@@ -148,5 +148,5 @@
     </gazebo>
     <gazebo reference="gripper_finger_left">
-        <material>Gazebo/Orange</material>
+        <material>Gazebo/Trunk  </material>
         <gravity>true</gravity>
         <ode>
@@ -160,5 +160,5 @@
     </gazebo>
     <gazebo reference="gripper_finger_right">
-        <material>Gazebo/Orange</material>
+        <material>Gazebo/Trunk  </material>
         <gravity>true</gravity>
         <ode>

File: src/robot_model/urdf/robot_core.xacro (robot description, xacro)
@@ -65,5 +65,5 @@
     </link>
     <gazebo reference="chassis">
-        <material>Gazebo/Pink</material>
+        <material>Gazebo/Wood   </material>
     </gazebo>
     <!-- Wheel Link -->
@@ -85,5 +85,5 @@
     </link>
     <gazebo reference="front_left_wheel">
-        <material>Gazebo/Red</material>
+        <material>Gazebo/CloudySky </material>
     </gazebo>
     <link name="front_right_wheel">
@@ -104,5 +104,5 @@
     </link>
     <gazebo reference="front_right_wheel">
-        <material>Gazebo/Red</material>
+        <material>Gazebo/CloudySky </material>
     </gazebo>
     <link name="back_left_wheel">
@@ -123,5 +123,5 @@
     </link>
     <gazebo reference="back_left_wheel">
-        <material>Gazebo/Red</material>
+        <material>Gazebo/CloudySky </material>
     </gazebo>
     <link name="back_right_wheel">
@@ -142,5 +142,5 @@
     </link>
     <gazebo reference="back_right_wheel">
-        <material>Gazebo/Red</material>
+        <material>Gazebo/CloudySky </material>
     </gazebo>
     <!-- Wheel Joint -->
